Commit message: cleanup, racer launch file

File: urdf/src/racer_description/urdf/racer.urdf (robot description, URDF)
Before this commit: robot racer, 9 links, 8 joints
Joints:
- joint fixed: axis 0 -1 0 -> 0 0 0; limit lower=-1.7 upper=1.7 effort=10000.0 velocity=6.98131700798 -> lower=0 upper=0 effort=0.0 velocity=0; origin xyz=0 0 2.37 rpy=0.0 3.1415926536 3.1415926536 -> xyz=0 0 0 rpy=0.0 0.0 0.0; type prismatic -> fixed
