Commit message: working w/ pinocchio3-preview, with built-in casadi, to address issue of non-symmetric mass matrix in other library

File: urdf/src/racer_description/urdf/racer7.urdf (robot description, URDF)
Before this commit: robot racer7, 9 links, 8 joints
Links:
- link base_link: mass 6.215 -> 75.931
- link link_1: mass 5.46814182699 -> 22.4953
- link link_2: mass 3.4970386262 -> 23.396
- link link_4: mass 1.62984418881 -> 13.0332
- link link_5: mass 0.805335362671 -> 4.03009
- link link_6: mass 0.073 -> 0.267
Joints:
- joint fixed: axis 0 -1 0 -> 0 0 0; limit lower=-1.7 upper=1.7 effort=10000.0 velocity=6.98131700798 -> lower=0 upper=0 effort=0.0 velocity=0; origin xyz=0 0 2.37 rpy=0.0 3.1415926536 3.1415926536 -> xyz=0 0 0 rpy=0.0 0.0 0.0; type prismatic -> fixed
- joint head_swivel: origin xyz=0.0 0.0 0.1895 rpy=0 0 0 -> xyz=0.0 0.0 0.430 rpy=0 0 0
- joint joint_2: origin xyz=0.05 0.0 0.1755 rpy=0.0 1.57 0.0 -> xyz=0.05 0.0 0.590 rpy=0.0 1.57 0.0
- joint joint_3: origin xyz=0.0 0.0 0.37 rpy=0.0 -1.57 0.0 -> xyz=0.0 0.0 0.684 rpy=0.0 -1.57 0.0

Commit message: fix some array formatting errors; mostly stable in joint space now

File: urdf/src/racer_description/urdf/racer7.urdf (robot description, URDF)
Before this commit: robot racer7, 9 links, 8 joints
Links:
- link link_5: mass 4.03009 -> 6.03009
- link link_6: mass 0.267 -> 6.267

Commit message: fixed racer urdf file, kinematics seems OK

File: urdf/src/racer_description/urdf/racer7.urdf (robot description, URDF)
Before this commit: robot racer7, 9 links, 8 joints
Joints:
- joint gripper_fixed: origin xyz=-0.101962 0.0 0.46533 rpy=3.1415926536 0.0 0.0 -> xyz=0.0 0.0 0.0 rpy=0.0 0.0 0.0
- joint joint_2: axis 0 -1  0 -> 0 1 0; origin xyz=0.05 0.0 0.590 rpy=0.0 1.57 0.0 -> xyz=0.150 0.0 0.0 rpy=0.0 0.0 0.0
- joint joint_3: axis 0 -1  0 -> 0 -1 0; origin xyz=0.0 0.0 0.684 rpy=0.0 -1.57 0.0 -> xyz=0.0 0.0 0.590 rpy=0.0 0.0 0.0
- joint joint_4: axis 0  0 -1 -> 0 0 -1; origin xyz=-0.049998 0 0.121 rpy=0 0 0 -> xyz=-0.130 0 0 rpy=0 0 0
- joint joint_5: axis 0 -1  0 -> 0 1 0; origin xyz=0 0 0.26494 rpy=0 0 0 -> xyz=0 0 0.684 rpy=0 0 0
- joint joint_6: axis 0  0 -1 -> 0 0 -1; origin xyz=0 0 0.0665 rpy=0 0 0 -> xyz=0.0 0.0 0.1 rpy=0 0 0

Commit message: Tuned regularizatoin on param_fit

File: urdf/src/racer_description/urdf/racer7.urdf (robot description, URDF)
Before this commit: robot racer7, 9 links, 8 joints
Joints:
- joint head_swivel: axis 0  0  1 -> 0  0  -1
