Commit message: trying to fix URDF, still a couple issues to check (joint 2 seems to be about wrong axis?)

File: urdf/src/racer_description/urdf/.ipynb_checkpoints/racer-checkpoint.urdf (robot description, URDF)
Before this commit: robot racer7, 9 links, 8 joints
Links:
- link base_link: mass 75.931 -> 6.215; geometry collision mesh filename=package://racer_description/mesh/base_link.STL; visual mesh filename=package://racer_description/mesh/base_link.STL
- link gripper: geometry collision mesh filename=package://racer_description/mesh/gripper_v2.STL; visual mesh filename=package://racer_description/mesh/gripper_v2.STL
- link link_1: mass 22.4953 -> 5.46814182699; geometry collision mesh filename=package://racer_description/mesh/link_1.STL; visual mesh filename=package://racer_description/mesh/link_1.STL
- link link_2: mass 23.396 -> 3.4970386262; geometry collision mesh filename=package://racer_description/mesh/link_2.STL; visual mesh filename=package://racer_description/mesh/link_2.STL
- link link_3: geometry collision mesh filename=package://racer_description/mesh/link_3.STL; visual mesh filename=package://racer_description/mesh/link_3.STL
- link link_4: mass 13.0332 -> 1.62984418881; geometry collision mesh filename=package://racer_description/mesh/link_4.STL; visual mesh filename=package://racer_description/mesh/link_4.STL
- link link_5: mass 6.03009 -> 0.805335362671; geometry collision mesh filename=package://racer_description/mesh/link_5.STL; visual mesh filename=package://racer_description/mesh/link_5.STL
- link link_6: mass 6.267 -> 0.073; geometry collision mesh filename=package://racer_description/mesh/link_6.STL; visual mesh filename=package://racer_description/mesh/link_6.STL
Joints:
- joint head_swivel: origin xyz=0.0 0.0 0.430 rpy=0 0 0 -> xyz=0.0 0.0 0.1895 rpy=0 0 0
- joint joint_2: origin xyz=0.05 0.0 0.590 rpy=0.0 1.57 0.0 -> xyz=0.05 0.0 0.1755 rpy=0.0 1.57 0.0
- joint joint_3: origin xyz=0.0 0.0 0.684 rpy=0.0 -1.57 0.0 -> xyz=0.0 0.0 0.37 rpy=0.0 -1.57 0.0
